File: CosmosBoard/sensors.kicad_sch (KiCad schematic)
At the start: 88 parts, among them J10 Conn_01x04, J11 Conn_01x06, J13 Conn_01x08, J14 Conn_01x07, J15 Conn_01x05, J16 Conn_01x04, J17 Conn_01x03, J18 Conn_01x03, J19 Conn_01x04, J20 Conn_01x02, J5 Conn_01x02, J6 Conn_01x02, J7 Conn_01x02, J8 Conn_01x02, J9 Conn_01x08, M1 Motor_Servo, M2 Motor_Servo, M3 Motor_Servo, M4 Motor_Servo, SW10 SW_Push_SPDT, SW11 SW_Push_SPDT, SW3 SW_Push, SW4 SW_Push, SW5 SW_Push, SW6 SW_Push, SW7 RotaryEncoder_Switch, SW8 SW_Push_SPDT, SW9 SW_Push_SPDT, U2 BNO055, U4 BMP280, U5 E32-915T30S, U6 AMS1117-3.3, U7 AMS1117-3.3, Y2 32.768

Commit message: alligns
Parts:
- removed J11: Conn_01x06, Connector_PinHeader_2.54mm:PinHeader_1x06_P2.54mm_Vertical, symbol Connector_Generic:Conn_01x06
- added J11: Conn_01x05, Connector_PinHeader_2.54mm:PinHeader_1x05_P2.54mm_Vertical, symbol Connector_Generic:Conn_01x05
Connections:
- net AUX: now also J11.5 (Pin_5)
- net at U5.4 (TXD): now also J11.4 (Pin_4)
- net at U5.3 (RXD): now also J11.3 (Pin_3)
- net at U5.2 (M1): now also J11.2 (Pin_2)
- net at U5.1 (M0): now also J11.1 (Pin_1)
- net ANT: no longer names the net of U5.18 (ANT)
- no-connect marks 4 -> 5
Changed lines of the file:
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@@
 		(at 196.85 172.72)
 	)
+	(no_connect
+		(at 257.81 170.18)
+	)
 	(wire
 		(pts
@@
 	(wire
 		(pts
+			(xy 298.45 165.1) (xy 298.45 167.64)
+		)
+		(stroke
+			(width 0)
+			(type default)
+		)
+	)
+	(wire
+		(pts
 			(xy 369.57 222.25) (xy 373.38 222.25)
 		)
@@
 	(wire
 		(pts
-			(xy 293.37 167.64) (xy 293.37 165.1)
+			(xy 182.88 49.53) (xy 182.88 45.72)
 		)
 		(stroke
@@
 	(wire
 		(pts
-			(xy 182.88 49.53) (xy 182.88 45.72)
+			(xy 208.28 53.34) (xy 203.2 53.34)
 		)
 		(stroke
@@
 	(wire
 		(pts
-			(xy 208.28 53.34) (xy 203.2 53.34)
+			(xy 293.37 165.1) (xy 298.45 165.1)
 		)
 		(stroke
@@
 	(wire
 		(pts
-			(xy 309.88 167.64) (xy 293.37 167.64)
+			(xy 298.45 167.64) (xy 309.88 167.64)
 		)
 		(stroke
@@
 		)
 	)
-	(label "ANT"
-		(at 309.88 162.56 180)
-		(fields_autoplaced yes)
-		(effects
-			(font
-				(size 1.27 1.27)
-			)
-			(justify right bottom)
-		)
-	)
 	(label "BNO_08x_CS"
 		(at 288.29 86.36 0)
@@
 		)
 	)
-	(label "ANT"
-		(at 257.81 170.18 180)
-		(fields_autoplaced yes)
-		(effects
-			(font
-				(size 1.27 1.27)
-			)
-			(justify right bottom)
-		)
-	)
 	(label "SPI_2_MISO_I2C_SDA_UART_TX"
 		(at 276.86 81.28 0)
@@
 	)
 	(symbol
-		(lib_id "Connector_Generic:Conn_01x06")
-		(at 314.96 170.18 0)
-		(mirror x)
-		(unit 1)
-		(exclude_from_sim no)
-		(in_bom yes)
-		(on_board yes)
-		(dnp no)
-		(fields_autoplaced yes)
-		(property "Reference" "J11"
-			(at 314.96 156.21 0)
-			(effects
-				(font
-					(size 1.27 1.27)
-				)
-			)
-		)
-		(property "Value" "Conn_01x06"
-			(at 314.96 158.75 0)
-			(effects
-				(font
-					(size 1.27 1.27)
-				)
-			)
-		)
-		(property "Footprint" "Connector_PinHeader_2.54mm:PinHeader_1x06_P2.54mm_Vertical"
-			(at 314.96 170.18 0)
-			(effects
-				(font
-					(size 1.27 1.27)
-				)
-				(hide yes)
-			)
-		)
-		(property "Datasheet" "~"
-			(at 314.96 170.18 0)
-			(effects
-				(font
-					(size 1.27 1.27)
-				)
-				(hide yes)
-			)
-		)
-		(property "Description" "Generic connector, single row, 01x06, script generated (kicad-library-utils/schlib/autogen/connector/)"
-			(at 314.96 170.18 0)
-			(effects
-				(font
-					(size 1.27 1.27)
-				)
-				(hide yes)
-			)
-		)
-		(pin "1"
-		)
-		(pin "5"
-		)
-		(pin "4"
-		)
-		(pin "6"
-		)
-		(pin "2"
-		)
-		(pin "3"
-		)
-		(instances
-			(project "CosmosBoard"
-				(path "/8edaa023-92cc-4c4a-9f01-71d27077a029/8249c00b-69f6-4519-9811-4d5dc3fe2a3c"
-					(reference "J11")
-					(unit 1)
-				)
-			)
-		)
-	)
-	(symbol
 		(lib_id "Device:R")
 		(at 273.05 210.82 0)
@@
 					(unit 1)
 				)
+			)
+		)
+	)
+	(symbol
+		(lib_id "Connector_Generic:Conn_01x05")
+		(at 314.96 170.18 0)
+		(unit 1)
+		(exclude_from_sim no)
+		(in_bom yes)
+		(on_board yes)
+		(dnp no)
+		(property "Reference" "J11"
+			(at 313.182 162.052 0)
+			(effects
+				(font
+					(size 1.27 1.27)
+				)
+				(justify left)
+			)
+		)
+		(property "Value" "Conn_01x05"
+			(at 309.118 178.562 0)
+			(effects
+				(font
+					(size 1.27 1.27)
+				)
+				(justify left)
+			)
+		)
+		(property "Footprint" "Connector_PinHeader_2.54mm:PinHeader_1x05_P2.54mm_Vertical"
+			(at 314.96 170.18 0)
+			(effects
+				(font
+					(size 1.27 1.27)
+				)
+				(hide yes)
+			)
+		)
+		(property "Datasheet" "~"
+			(at 314.96 170.18 0)
+			(effects
+				(font
+					(size 1.27 1.27)
+				)
+				(hide yes)
+			)
+		)
+		(property "Description" "Generic connector, single row, 01x05, script generated (kicad-library-utils/schlib/autogen/connector/)"
+			(at 314.96 170.18 0)
+			(effects
+				(font
+					(size 1.27 1.27)
+				)
+				(hide yes)
+			)
+		)
+		(pin "2"
+		)
+		(pin "1"
+		)
+		(pin "3"
+		)
+		(pin "4"
+		)
+		(pin "5"
+		)
+		(instances
+			(project "CosmosBoard"
+				(path "/8edaa023-92cc-4c4a-9f01-71d27077a029/8249c00b-69f6-4519-9811-4d5dc3fe2a3c"
+					(reference "J11")
+					(unit 1)
+				)

Commit message: pre-final
Parts:
- RV1, RV2, RV3: footprint Potentiometer_THT:Potentiometer_Omeg_PC16BU_Vertical -> Potentiometer_THT:Potentiometer_TT_P0915N
Changed lines of the file:
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@@
 			)
 		)
-		(property "Footprint" "Potentiometer_THT:Potentiometer_Omeg_PC16BU_Vertical"
+		(property "Footprint" "Potentiometer_THT:Potentiometer_TT_P0915N"
 			(at 119.38 35.56 0)
 			(effects
@@
 			)
 		)
-		(property "Footprint" "Potentiometer_THT:Potentiometer_Omeg_PC16BU_Vertical"
+		(property "Footprint" "Potentiometer_THT:Potentiometer_TT_P0915N"
 			(at 93.98 35.56 0)
 			(effects
@@
 			)
 		)
-		(property "Footprint" "Potentiometer_THT:Potentiometer_Omeg_PC16BU_Vertical"
+		(property "Footprint" "Potentiometer_THT:Potentiometer_TT_P0915N"
 			(at 106.68 35.56 0)
 			(effects
